File: KiCad Projects/BMW E30 VFL SI Indicator V2/BMW E30 VFL SI Indicator V2.kicad_pcb (KiCad board)
At the start: 2 copper layers, 58 x 32.4 mm, 13 parts, among them J1 Conn_01x13_Socket

Commit message: Add files via upload
Parts:
- moved J1 1.24 mm to (135.1, 90.4)
Routing:
- net Net-(D1-A): track 92.0 -> 80.1 mm
- net Net-(J1-GND_BULB): track 60.5 -> 58.4 mm
- net Net-(D3-K): track 9.42 -> 7.76 mm
- net Net-(D5-K): track 6.67 -> 5.38 mm
- net Net-(D4-K): track 7.05 -> 5.81 mm
- net Net-(D8-K): track 14.7 -> 13.6 mm
- net Net-(D9-K): track 18.6 -> 17.4 mm
- net Net-(J1-BULB_INSPECTION): track 63.7 -> 62.6 mm
- net Net-(D2-K): track 12.3 -> 11.2 mm
- net Net-(D7-K): track 11.0 -> 10.1 mm
- net Net-(D1-K): track 15.7 -> 14.8 mm
Other:
- board text added: "BMW E30 VFL VDO SI LIGHTS"
- board text added: "F. GMEINER 06/24 V2.1"
- board text removed: "BMW E30 VVFL VDO SI LIGHTS"
- board text removed: "F. GMEINER 06/24 V2.0"
